Commit message: Implemented example_01

File: robot.urdf (robot description, URDF)
Before this commit: robot xamla_motion_examples, 26 links, 25 joints
Links:
- added link cell_body, mass 1.0; collision mesh filename=package://part_sda10d_cell/collision/cell.stl scale=1.00 1.00 1.00; visual mesh filename=package://part_sda10d_cell/visual/cell.dae scale=1.00 1.00 1.00
- added link cell_tool0
Joints:
- added joint cell_body_to_tool0: type fixed, parent cell_body, child cell_tool0, origin xyz=0 0 0.16 rpy=0 0 0
- added joint world_to_cell_body: type fixed, parent world, child cell_body, origin xyz=0 0 0 rpy=0 0 0

File: robotModel/main.xacro (robot description, xacro)
@@ -11,3 +11,7 @@
     <origin xyz="0 0 0" rpy="0 0 0" />
   </xacro:part_wsg50>
+  <xacro:include filename="part_sda10d_cell/sda10d_cell.xacro" xamla:xref="object$sda10d_cell_1" />
+  <xacro:sda10d_cell xamla:xref="object$sda10d_cell_1" prefix="" parent="world">
+    <origin xyz="0 0 0" rpy="0 0 0" />
+  </xacro:sda10d_cell>
 </robot>

Commit message: Generate a grid of poses out of a pose, let the robot pick and place every pose

File: robot.urdf (robot description, URDF)
Before this commit: robot xamla_motion_examples, 28 links, 27 joints
Joints:
- joint _base_joint_gripper_right: limit lower=0.0027 upper=0.055 effort=80.0 velocity=0.42 -> lower=0.0028 upper=0.0549 effort=80.0 velocity=0.42
- joint arm_left_joint_1_s: limit lower=-3.13 upper=3.13 effort=0 velocity=2.95 -> lower=-3.0986 upper=3.0986 effort=0 velocity=2.95
- joint arm_left_joint_2_l: limit lower=-1.90 upper=1.90 effort=0 velocity=2.95 -> lower=-1.8809 upper=1.8809 effort=0 velocity=2.95
- joint arm_left_joint_3_e: limit lower=-2.95 upper=2.95 effort=0 velocity=2.95 -> lower=-2.9204 upper=2.9204 effort=0 velocity=2.95
- joint arm_left_joint_4_u: limit lower=-2.36 upper=2.36 effort=0 velocity=2.95 -> lower=-2.3362999999999996 upper=2.3362999999999996 effort=0 velocity=2.95
- joint arm_left_joint_5_r: limit lower=-3.13 upper=3.13 effort=0 velocity=3.48 -> lower=-3.0986 upper=3.0986 effort=0 velocity=3.48
- joint arm_left_joint_6_b: limit lower=-1.90 upper=1.90 effort=0 velocity=3.48 -> lower=-1.8809 upper=1.8809 effort=0 velocity=3.48
- joint arm_left_joint_7_t: limit lower=-3.13 upper=3.13 effort=0 velocity=6.97 -> lower=-3.0986 upper=3.0986 effort=0 velocity=6.97
- joint arm_right_joint_1_s: limit lower=-3.13 upper=3.13 effort=0 velocity=2.95 -> lower=-3.0986 upper=3.0986 effort=0 velocity=2.95
- joint arm_right_joint_2_l: limit lower=-1.90 upper=1.90 effort=0 velocity=2.95 -> lower=-1.8809 upper=1.8809 effort=0 velocity=2.95
- joint arm_right_joint_3_e: limit lower=-2.95 upper=2.95 effort=0 velocity=2.95 -> lower=-2.9204 upper=2.9204 effort=0 velocity=2.95
- joint arm_right_joint_4_u: limit lower=-2.36 upper=2.36 effort=0 velocity=2.95 -> lower=-2.3362999999999996 upper=2.3362999999999996 effort=0 velocity=2.95
- joint arm_right_joint_5_r: limit lower=-3.13 upper=3.13 effort=0 velocity=3.48 -> lower=-3.0986 upper=3.0986 effort=0 velocity=3.48
- joint arm_right_joint_6_b: limit lower=-1.90 upper=1.90 effort=0 velocity=3.48 -> lower=-1.8809 upper=1.8809 effort=0 velocity=3.48
- joint arm_right_joint_7_t: limit lower=-3.13 upper=3.13 effort=0 velocity=6.97 -> lower=-3.0986 upper=3.0986 effort=0 velocity=6.97
- joint torso_joint_b1: limit lower=-2.9570 upper=2.9570 effort=100 velocity=2.26 -> lower=-2.82833 upper=2.82833 effort=100 velocity=2.26
- joint torso_joint_b2: limit lower=-2.9570 upper=2.9570 effort=100 velocity=2.26 -> lower=-2.82833 upper=2.82833 effort=100 velocity=2.26

Commit message: Added offset for endeffecor and adjusted the examples

File: robot.urdf (robot description, URDF)
Before this commit: robot xamla_motion_examples, 28 links, 27 joints
Links:
- added link tcp_link_left
- added link tcp_link_right
Joints:
- added joint tcp_joint_left_F: type fixed, parent arm_left_link_tool0, child tcp_link_left, origin xyz=0.0 0.000 0.09 rpy=0 0 0
- added joint tcp_joint_right_F: type fixed, parent arm_right_link_tool0, child tcp_link_right, origin xyz=0.0 0.000 0.09 rpy=0 0 0

File: robotModel/main.xacro (robot description, xacro)
@@ -3,4 +3,16 @@
   <xacro:property name="pi" value="3.1415926535897931" />
   <link name="world" />
+  <link name="tcp_link_left" />
+  <joint name="tcp_joint_left_F" type="fixed">
+    <child link="tcp_link_left" />
+    <parent link="arm_left_link_tool0" />
+    <origin xyz="0.0 0.000 0.09" rpy="0 0 0" />
+  </joint>
+  <link name="tcp_link_right" />
+  <joint name="tcp_joint_right_F" type="fixed">
+    <child link="tcp_link_right" />
+    <parent link="arm_right_link_tool0" />
+    <origin xyz="0.0 0.000 0.09" rpy="0 0 0" />
+  </joint>
   <xacro:include filename="part_motoman_sda10f/sda10f_macro.xacro" xamla:xref="yaskawa$motoman_sda10f_1" />
   <xacro:motoman_sda10f xamla:xref="yaskawa$motoman_sda10f_1" prefix="" parent="world">
